File: hardware/rtc_xiao_esp32s3.kicad_pcb (KiCad board)
At the start: 4 copper layers, 17.5 x 21 mm, 24 parts, among them J1 +5V, J2 GND, J3 SCL, J4 SDA, J5 CLKOUT, J6 NINT, U1 RV-3028-C8

Commit message: pcb update
Parts:
- added REF**: PUTM_logo, PUTM_logo:PUTM_logo, B.Cu at (122.5, 104.5)
Other:
- board text added: "RTC for XIAO ESP32S3"

Commit message: minor changes
Parts:
- U1: footprint Samacsys:RV3028C832768kHz1PPMTAQC -> Xiao RTC:RV3028C832768kHz1PPMTAQC
